Commit message: chore: trying to fix frames

File: slam_bot/urdf/slam_bot.xacro (robot description, xacro)
@@ -4,9 +4,4 @@
   <xacro:include filename="$(find slam_bot)/urdf/slam_bot.gazebo"/>
   <link name="robot_footprint"></link>
-  <joint name="robot_footprint_joint" type="fixed">
-    <origin xyz="0 0 0" rpy="0 0 0" />
-    <parent link="robot_footprint"/>
-    <child link="chassis" />
-  </joint>
   <!-- Chassis Link -->
   <link name='chassis'>
@@ -136,5 +131,5 @@
   </link>
   <!-- Camera Link -->
-  <link name="camera_link">
+  <link name="camera">
     <inertial>
       <mass value="0.1"/>
@@ -187,4 +182,9 @@
   </link>
   <!-- Joints -->
+  <joint name="robot_footprint_joint" type="fixed">
+    <origin xyz="0 0 0" rpy="0 0 0" />
+    <parent link="robot_footprint"/>
+    <child link="chassis" />
+  </joint>
   <joint type="continuous" name="left_wheel_hinge">
     <origin xyz="0 0.25 0" rpy="0 0 0"/>
@@ -203,9 +203,15 @@
     <joint_properties damping="1.0" friction="1.0"/>
   </joint>
-  <joint type="fixed" name="camera_joint">
+  <joint type="fixed" name="camera_link">
     <origin xyz="0.25 0 0" rpy="0 0 0"/>
-    <child link="camera_link"/>
-    <parent link="chassis"/>
-  </joint>
+    <child link="camera"/>
+    <parent link="chassis"/>
+  </joint>
+  <joint name="camera_joint" type="fixed">
+      <origin xyz="0 0 0" rpy="-1.5707 0 -1.5707"/>
+      <parent link="camera"/>
+      <child link="camera_rgbd_frame"/>
+  </joint>
+  <link name="camera_rgbd_frame"/>
   <joint type="fixed" name="hokuyo_joint">
     <origin xyz="0.0 0 0.1" rpy="0 0 0"/>

Commit message: feat: slam_bot 3D-mapping

File: slam_bot/urdf/slam_bot.xacro (robot description, xacro)
@@ -176,5 +176,5 @@
     <collision>
       <geometry>
-        <box size="0.1 0.1 0.1"/>
+        <box size="0.2 0.2 0.2"/>
       </geometry>
       <origin xyz="0 0 0" rpy="0 0 0"/>
@@ -215,5 +215,5 @@
   <link name="camera_rgbd_frame"/>
   <joint type="fixed" name="hokuyo_joint">
-    <origin xyz="0.0 0 0.1" rpy="0 0 0"/>
+    <origin xyz="0.0 0 0.2" rpy="0 0 0"/>
     <child link="hokuyo"/>
     <parent link="chassis"/>

Commit message: fix: laser scanner works
modified the gazebo plug-in to gpu version.

File: slam_bot/urdf/slam_bot.xacro (robot description, xacro)
@@ -34,5 +34,5 @@
       <origin xyz="-0.15 0 -0.05" rpy=" 0 0 0"/>
       <geometry>
-        <sphere radius="0.05"/>
+        <sphere radius="0.0499"/>
       </geometry>
       <surface>
@@ -50,5 +50,5 @@
       <origin xyz="-0.15 0 -0.05" rpy=" 0 0 0"/>
       <geometry>
-        <sphere radius="0.05"/>
+        <sphere radius="0.0499"/>
       </geometry>
     </visual>
@@ -56,5 +56,5 @@
       <origin xyz="0.15 0 -0.05" rpy=" 0 0 0"/>
       <geometry>
-        <sphere radius="0.05"/>
+        <sphere radius="0.0499"/>
       </geometry>
       <surface>
@@ -72,5 +72,5 @@
       <origin xyz="0.15 0 -0.05" rpy=" 0 0 0"/>
       <geometry>
-        <sphere radius="0.05"/>
+        <sphere radius="0.0499"/>
       </geometry>
     </visual>
@@ -176,5 +176,5 @@
     <collision>
       <geometry>
-        <box size="0.2 0.2 0.2"/>
+        <box size="0.1 0.1 0.075"/>
       </geometry>
       <origin xyz="0 0 0" rpy="0 0 0"/>
@@ -204,5 +204,5 @@
   </joint>
   <joint type="fixed" name="camera_link">
-    <origin xyz="0.25 0 0" rpy="0 0 0"/>
+    <origin xyz="0.2 0 0" rpy="0 0 0"/>
     <child link="camera"/>
     <parent link="chassis"/>
@@ -215,5 +215,5 @@
   <link name="camera_rgbd_frame"/>
   <joint type="fixed" name="hokuyo_joint">
-    <origin xyz="0.0 0 0.2" rpy="0 0 0"/>
+    <origin xyz="0.15 0 0.1" rpy="0 0 0"/>
     <child link="hokuyo"/>
     <parent link="chassis"/>
